File: BMS_stack_monitor.sch (KiCad schematic (older format))
At the start: 17 parts, among them J6 JST_XH-13, U3 LTC6803-3

Commit message: HW 0.2 finalized schematic and pcb files, BOM needs to be checked
Lots of major and little problems fixed found in the 0.1

Major changes:
-LTC6803-3 footprint changed to it's correct one
-Boost converter layout and capacitor optimization
-MCU switched from STM32F070CBT6 to ultra low power STM32L433CCT6 to improve sleep state power consumption
-Button/LED + Comms connectors switched from THT JST-XH to SMD JST-PH
-CAN-bus support added
-Changed power regulator setup for "always on"

Minor changes:
-Changed cell balance resistor sizes from 0603 to 0402 in order to get a bit more breathing room during soldering
-External oscillator removed from MCU, because new one has everything available internally
-Comms connector has USART or CAN available via solder bridges
-Sense resistors switched to higher resistance ones to lower deep sleep standby current
-etc.
Parts:
- C11, C12: MFG EMK107BJ225KA-T -> ANY; TempCo. (none) -> X5R
- C13, C43: MFG CL10B104KC8NNNC -> ANY; TempCo. (none) -> X7R
- R19, R24: MFG RC0603FR-074K7L -> ANY; Tol. (none) -> 1%
- R21, R23, R25: MFG RC0603FR-071ML -> ANY; Tol. (none) -> 1%
- R26, R77: MFG RC0603FR-07120RL -> ANY; Tol. (none) -> 1%
- R27: footprint Resistors_SMD:R_0603 -> Resistors_SMD:R_0402; MFG RC0603FR-07120RL -> ANY; Tol. (none) -> 1%
- U3: footprint Housings_SSOP:TSSOP-44_4.4x11.2mm_Pitch0.5mm -> Custom_footprints:FSOP-44_5.3x13.0mm_Pitch0.5mm
Changed lines of the file:
@@
 LIBS:valves
 LIBS:Custom_comp_lib
-LIBS:FlexiBMS_01-cache
+LIBS:FlexiBMS-cache
 EELAYER 25 0
 EELAYER END
@@
 Title "FlexiBMS"
 Date "2018-02-22"
-Rev "0.1"
+Rev "0.2"
 Comp "SiMoS MCmuffin / Simo Sihvonen"
 Comment1 ""
@@
 F 0 "U3" H 3500 6250 60  0000 C CNN
 F 1 "LTC6803-3" H 3500 1850 60  0000 C CNN
-F 2 "Housings_SSOP:TSSOP-44_4.4x11.2mm_Pitch0.5mm" H 3500 4100 60  0001 C CNN
+F 2 "Custom_footprints:FSOP-44_5.3x13.0mm_Pitch0.5mm" H 3500 4100 60  0001 C CNN
 F 3 "" H 3500 4100 60  0001 C CNN
 F 4 "LTC6803IG-3#PBF" H 3500 4100 60  0001 C CNN "MFG"
@@
 F 2 "Capacitors_SMD:C_0603" H 1788 4900 50  0001 C CNN
 F 3 "" H 1750 5050 50  0001 C CNN
-F 4 "EMK107BJ225KA-T" H 1750 5050 60  0001 C CNN "MFG"
+F 4 "ANY" H 1750 5050 60  0001 C CNN "MFG"
+F 5 "X5R" H 1750 5050 60  0001 C CNN "TempCo."
 	1    1750 5050
 	1    0    0    -1
@@
 F 2 "Capacitors_SMD:C_0603" H 2188 4900 50  0001 C CNN
 F 3 "" H 2150 5050 50  0001 C CNN
-F 4 "EMK107BJ225KA-T" H 2150 5050 60  0001 C CNN "MFG"
+F 4 "ANY" H 2150 5050 60  0001 C CNN "MFG"
+F 5 "X5R" H 2150 5050 60  0001 C CNN "TempCo."
 	1    2150 5050
 	1    0    0    -1
@@
 F 2 "Resistors_SMD:R_0603" V 4230 1450 50  0001 C CNN
 F 3 "" H 4300 1450 50  0001 C CNN
-F 4 "RC0603FR-07120RL" V 4300 1450 60  0001 C CNN "MFG"
+F 4 "ANY" V 4300 1450 60  0001 C CNN "MFG"
+F 5 "1%" V 4300 1450 60  0001 C CNN "Tol."
 	1    4300 1450
 	1    0    0    -1
@@
 F 2 "Capacitors_SMD:C_0603" H 4138 1600 50  0001 C CNN
 F 3 "" H 4100 1750 50  0001 C CNN
-F 4 "CL10B104KC8NNNC" H 4100 1750 60  0001 C CNN "MFG"
+F 4 "ANY" H 4100 1750 60  0001 C CNN "MFG"
+F 5 "X7R" H 4100 1750 60  0001 C CNN "TempCo."
 	1    4100 1750
 	0    -1   -1   0
@@
 F 2 "Resistors_SMD:R_0603" V 2330 3250 50  0001 C CNN
 F 3 "" H 2400 3250 50  0001 C CNN
-F 4 "RC0603FR-071ML" V 2400 3250 60  0001 C CNN "MFG"
+F 4 "ANY" V 2400 3250 60  0001 C CNN "MFG"
+F 5 "1%" V 2400 3250 60  0001 C CNN "Tol."
 	1    2400 3250
 	1    0    0    -1
@@
 F 2 "Resistors_SMD:R_0603" V 2130 3250 50  0001 C CNN
 F 3 "" H 2200 3250 50  0001 C CNN
-F 4 "RC0603FR-074K7L" V 2200 3250 60  0001 C CNN "MFG"
+F 4 "ANY" V 2200 3250 60  0001 C CNN "MFG"
+F 5 "1%" V 2200 3250 60  0001 C CNN "Tol."
 	1    2200 3250
 	1    0    0    -1
@@
 F 2 "Resistors_SMD:R_0603" V 1930 3250 50  0001 C CNN
 F 3 "" H 2000 3250 50  0001 C CNN
-F 4 "RC0603FR-071ML" V 2000 3250 60  0001 C CNN "MFG"
+F 4 "ANY" V 2000 3250 60  0001 C CNN "MFG"
+F 5 "1%" V 2000 3250 60  0001 C CNN "Tol."
 	1    2000 3250
 	1    0    0    -1
@@
 F 2 "Resistors_SMD:R_0603" V 1730 3250 50  0001 C CNN
 F 3 "" H 1800 3250 50  0001 C CNN
-F 4 "RC0603FR-071ML" V 1800 3250 60  0001 C CNN "MFG"
+F 4 "ANY" V 1800 3250 60  0001 C CNN "MFG"
+F 5 "1%" V 1800 3250 60  0001 C CNN "Tol."
 	1    1800 3250
 	1    0    0    -1
@@
 	1450 3800 2800 3800
 $Comp
-L +3V3 #PWR033
+L +3V3 #PWR032
 U 1 1 5A82AA4B
 P 2000 2950
-F 0 "#PWR033" H 2000 2800 50  0001 C CNN
+F 0 "#PWR032" H 2000 2800 50  0001 C CNN
 F 1 "+3V3" H 2000 3090 50  0000 C CNN
 F 2 "" H 2000 2950 50  0001 C CNN
@@
 F 2 "Resistors_SMD:R_0603" V 1930 4100 50  0001 C CNN
 F 3 "" H 2000 4100 50  0001 C CNN
-F 4 "RC0603FR-074K7L" V 2000 4100 60  0001 C CNN "MFG"
+F 4 "ANY" V 2000 4100 60  0001 C CNN "MFG"
+F 5 "1%" V 2000 4100 60  0001 C CNN "Tol."
 	1    2000 4100
 	0    1    1    0
@@
 F 0 "R27" V 6230 6800 50  0000 C CNN
 F 1 "120R" V 6150 6800 50  0000 C CNN
-F 2 "Resistors_SMD:R_0603" V 6080 6800 50  0001 C CNN
+F 2 "Resistors_SMD:R_0402" V 6080 6800 50  0001 C CNN
 F 3 "" H 6150 6800 50  0001 C CNN
-F 4 "RC0603FR-07120RL" V 6150 6800 60  0001 C CNN "MFG"
+F 4 "ANY" V 6150 6800 60  0001 C CNN "MFG"
+F 5 "1%" V 6150 6800 60  0001 C CNN "Tol."
 	1    6150 6800
 	0    1    1    0
@@
 BAT+
 $Comp
-L GND #PWR034
+L GND #PWR033
 U 1 1 5A82AA5F
 P 2700 6550
-F 0 "#PWR034" H 2700 6300 50  0001 C CNN
+F 0 "#PWR033" H 2700 6300 50  0001 C CNN
 F 1 "GND" H 2700 6400 50  0000 C CNN
 F 2 "" H 2700 6550 50  0001 C CNN
@@
 Connection ~ 2700 6450
 $Comp
-L GND #PWR035
+L GND #PWR034
 U 1 1 5A82AA60
 P 3800 1300
-F 0 "#PWR035" H 3800 1050 50  0001 C CNN
+F 0 "#PWR034" H 3800 1050 50  0001 C CNN
 F 1 "GND" H 3800 1150 50  0000 C CNN
 F 2 "" H 3800 1300 50  0001 C CNN
@@
 $EndSheet
 $Comp
-L GND #PWR036
+L GND #PWR035
 U 1 1 5A85FF70
 P 1500 1250
-F 0 "#PWR036" H 1500 1000 50  0001 C CNN
+F 0 "#PWR035" H 1500 1000 50  0001 C CNN
 F 1 "GND" H 1500 1100 50  0000 C CNN
 F 2 "" H 1500 1250 50  0001 C CNN
@@
 $EndComp
 $Comp
-L +3V3 #PWR037
+L +3V3 #PWR036
 U 1 1 5A85FF76
 P 1400 1050
-F 0 "#PWR037" H 1400 900 50  0001 C CNN
+F 0 "#PWR036" H 1400 900 50  0001 C CNN
 F 1 "+3V3" H 1400 1190 50  0000 C CNN
 F 2 "" H 1400 1050 50  0001 C CNN
@@
 F 2 "Capacitors_SMD:C_0603" H 4938 6550 50  0001 C CNN
 F 3 "" H 4900 6700 50  0001 C CNN
-F 4 "CL10B104KC8NNNC" H 4900 6700 60  0001 C CNN "MFG"
+F 4 "ANY" H 4900 6700 60  0001 C CNN "MFG"
+F 5 "X7R" H 4900 6700 60  0001 C CNN "TempCo."
 	1    4900 6700
 	1    0    0    -1
 $EndComp
 $Comp
-L GND #PWR038
+L GND #PWR037
 U 1 1 5A8F2374
 P 4900 6950
-F 0 "#PWR038" H 4900 6700 50  0001 C CNN
+F 0 "#PWR037" H 4900 6700 50  0001 C CNN
 F 1 "GND" H 4900 6800 50  0000 C CNN
 F 2 "" H 4900 6950 50  0001 C CNN
@@
 F 2 "Resistors_SMD:R_0603" V 3430 6450 50  0001 C CNN
 F 3 "" H 3500 6450 50  0001 C CNN
-F 4 "RC0603FR-07120RL" V 3500 6450 60  0001 C CNN "MFG"
+F 4 "ANY" V 3500 6450 60  0001 C CNN "MFG"
+F 5 "1%" V 3500 6450 60  0001 C CNN "Tol."
 	1    3500 6450
 	0    1    1    0
@@
 Data
 89 50 4E 47 0D 0A 1A 0A 00 00 00 0D 49 48 44 52 00 00 02 F2 00 00 01 DF 08 02 00 00 00 BD 23 AB
-6E 00 00 00 03 73 42 49 54 08 08 08 DB E1 4F E0 00 00 00 09 70 48 59 73 00 00 0E C3 00 00 0E C3
-01 C7 6F A8 64 00 00 20 00 49 44 41 54 78 9C EC 9D 77 9C 1D 55 D9 C7 7F CF 39 67 EE DD 4D CF 26
+6E 00 00 00 03 73 42 49 54 08 08 08 DB E1 4F E0 00 00 00 09 70 48 59 73 00 00 0E 74 00 00 0E 74
+01 6B 24 B3 D6 00 00 20 00 49 44 41 54 78 9C EC 9D 77 9C 1D 55 D9 C7 7F CF 39 67 EE DD 4D CF 26
 94 34 08 01 95 8E D4 50 44 54 8A 08 AF 14 21 2A 82 28 A0 E0 8B 22 E8 4B 91 26 BC A2 80 20 16 14
 A4 84 22 16 9A 80 E2 2B 4D 04 41 41 11 88 84 96 40 42 09 24 84 96 BE D9 BD 77 E6 9C E7 79 FF 38
@@
 Data
 89 50 4E 47 0D 0A 1A 0A 00 00 00 0D 49 48 44 52 00 00 02 30 00 00 01 11 08 02 00 00 00 EA 8B 0A
-36 00 00 00 03 73 42 49 54 08 08 08 DB E1 4F E0 00 00 00 09 70 48 59 73 00 00 0E C3 00 00 0E C3
-01 C7 6F A8 64 00 00 20 00 49 44 41 54 78 9C EC 7D 77 BC 15 C5 F9 FE F3 CE CC EE 39 B7 70 E9 45
+36 00 00 00 03 73 42 49 54 08 08 08 DB E1 4F E0 00 00 00 09 70 48 59 73 00 00 0E 74 00 00 0E 74
+01 6B 24 B3 D6 00 00 20 00 49 44 41 54 78 9C EC 7D 77 BC 15 C5 F9 FE F3 CE CC EE 39 B7 70 E9 45
 04 51 69 52 AC 80 22 D8 C0 58 31 A2 C6 18 0D F6 12 7B 6F 31 6A EC 3D 26 B6 C4 34 A3 51 4C 6C B1
 C6 44 45 04 15 82 88 1D 54 50 10 E9 BD DC 76 CA EE CC FB FE FE 98 3D E7 1E AE 18 A3 31 BF AF 26
