File: BMS_stack_monitor.sch (KiCad schematic (older format))
At the start: 17 parts, among them J6 JST_XH-13, U3 LTC6803-3

Commit message: 0.2 HW files finalized and repo cleaned up.
-BOM is now up-to-date and available in .csv and .pdf formats
Parts:
- J6: MFG S13B-XH-A(LF)(SN) -> \"S13B-XH-A(LF)(SN)\"/\"B13B-XH-A(LF)(SN)\"
Changed lines of the file:
@@
 F 2 "Connectors_JST:JST_XH_S13B-XH-A_13x2.50mm_Angled" H 8450 3700 50  0001 C CNN
 F 3 "" H 8450 3700 50  0001 C CNN
-F 4 "S13B-XH-A(LF)(SN)" H 8450 3700 60  0001 C CNN "MFG"
+F 4 "\"S13B-XH-A(LF)(SN)\"/\"B13B-XH-A(LF)(SN)\"" H 8450 3700 60  0001 C CNN "MFG"
 	1    8450 3700
 	1    0    0    -1
