File: currentMeasuring.sch (KiCad schematic (older format))
At the start: 10 parts, among them U5 ISL28022

Commit message: HW 0.2 finalized schematic and pcb files, BOM needs to be checked
Lots of major and little problems fixed found in the 0.1

Major changes:
-LTC6803-3 footprint changed to it's correct one
-Boost converter layout and capacitor optimization
-MCU switched from STM32F070CBT6 to ultra low power STM32L433CCT6 to improve sleep state power consumption
-Button/LED + Comms connectors switched from THT JST-XH to SMD JST-PH
-CAN-bus support added
-Changed power regulator setup for "always on"

Minor changes:
-Changed cell balance resistor sizes from 0603 to 0402 in order to get a bit more breathing room during soldering
-External oscillator removed from MCU, because new one has everything available internally
-Comms connector has USART or CAN available via solder bridges
-Sense resistors switched to higher resistance ones to lower deep sleep standby current
-etc.
Parts:
- C30, C32, C33, C34: MFG CL10B104KC8NNNC -> ANY; TempCo. (none) -> X7R
- C31: MFG EMK107BJ225KA-T -> ANY; TempCo. (none) -> X5R
- R64, R65: MFG RC0603FR-0710RL -> ANY; Tol. (none) -> 1%
- R66: MFG KRL1632E-M-R010-F-T5 -> ANY; Power (none) -> 0.75W; Tol. (none) -> 1%
Changed lines of the file:
@@
 LIBS:valves
 LIBS:Custom_comp_lib
-LIBS:FlexiBMS_01-cache
+LIBS:FlexiBMS-cache
 EELAYER 25 0
 EELAYER END
@@
 Title "FlexiBMS"
 Date "2018-02-22"
-Rev "0.1"
+Rev "0.2"
 Comp "SiMoS MCmuffin / Simo Sihvonen"
 Comment1 ""
@@
 $EndComp
 $Comp
-L GND #PWR048
+L GND #PWR050
 U 1 1 5A8315EC
 P 4550 3400
-F 0 "#PWR048" H 4550 3150 50  0001 C CNN
+F 0 "#PWR050" H 4550 3150 50  0001 C CNN
 F 1 "GND" H 4550 3250 50  0000 C CNN
 F 2 "" H 4550 3400 50  0001 C CNN
@@
 $EndComp
 $Comp
-L +3V3 #PWR049
+L +3V3 #PWR051
 U 1 1 5A8315ED
 P 5400 4350
-F 0 "#PWR049" H 5400 4200 50  0001 C CNN
+F 0 "#PWR051" H 5400 4200 50  0001 C CNN
 F 1 "+3V3" H 5400 4490 50  0000 C CNN
 F 2 "" H 5400 4350 50  0001 C CNN
@@
 F 2 "Capacitors_SMD:C_0603" H 7138 3600 50  0001 C CNN
 F 3 "" H 7100 3750 50  0001 C CNN
-F 4 "CL10B104KC8NNNC" H 7100 3750 60  0001 C CNN "MFG"
+F 4 "ANY" H 7100 3750 60  0001 C CNN "MFG"
+F 5 "X7R" H 7100 3750 60  0001 C CNN "TempCo."
 	1    7100 3750
 	1    0    0    -1
@@
 I2C_SCL
 $Comp
-L GND #PWR050
+L GND #PWR052
 U 1 1 5A8315F0
 P 6300 5050
-F 0 "#PWR050" H 6300 4800 50  0001 C CNN
+F 0 "#PWR052" H 6300 4800 50  0001 C CNN
 F 1 "GND" H 6300 4900 50  0000 C CNN
 F 2 "" H 6300 5050 50  0001 C CNN
@@
 F 2 "Capacitors_SMD:C_0603" H 6338 4550 50  0001 C CNN
 F 3 "" H 6300 4700 50  0001 C CNN
-F 4 "EMK107BJ225KA-T" H 6300 4700 60  0001 C CNN "MFG"
+F 4 "ANY" H 6300 4700 60  0001 C CNN "MFG"
+F 5 "X5R" H 6300 4700 60  0001 C CNN "TempCo."
 	1    6300 4700
 	1    0    0    -1
@@
 F 2 "Resistors_SMD:R_0603" V 7330 3150 50  0001 C CNN
 F 3 "" H 7400 3150 50  0001 C CNN
-F 4 "RC0603FR-0710RL" V 7400 3150 60  0001 C CNN "MFG"
+F 4 "ANY" V 7400 3150 60  0001 C CNN "MFG"
+F 5 "1%" V 7400 3150 60  0001 C CNN "Tol."
 	1    7400 3150
 	0    1    1    0
@@
 F 2 "Resistors_SMD:R_0603" V 7330 3550 50  0001 C CNN
 F 3 "" H 7400 3550 50  0001 C CNN
-F 4 "RC0603FR-0710RL" V 7400 3550 60  0001 C CNN "MFG"
+F 4 "ANY" V 7400 3550 60  0001 C CNN "MFG"
+F 5 "1%" V 7400 3550 60  0001 C CNN "Tol."
 	1    7400 3550
 	0    1    1    0
@@
 F 2 "Capacitors_SMD:C_0603" H 7138 2800 50  0001 C CNN
 F 3 "" H 7100 2950 50  0001 C CNN
-F 4 "CL10B104KC8NNNC" H 7100 2950 60  0001 C CNN "MFG"
+F 4 "ANY" H 7100 2950 60  0001 C CNN "MFG"
+F 5 "X7R" H 7100 2950 60  0001 C CNN "TempCo."
 	1    7100 2950
 	1    0    0    -1
 $EndComp
 $Comp
-L GND #PWR051
+L GND #PWR053
 U 1 1 5A8315F5
 P 7100 3950
-F 0 "#PWR051" H 7100 3700 50  0001 C CNN
+F 0 "#PWR053" H 7100 3700 50  0001 C CNN
 F 1 "GND" H 7100 3800 50  0000 C CNN
 F 2 "" H 7100 3950 50  0001 C CNN
@@
 $EndComp
 $Comp
-L GND #PWR052
+L GND #PWR054
 U 1 1 5A8315F6
 P 6850 2850
-F 0 "#PWR052" H 6850 2600 50  0001 C CNN
+F 0 "#PWR054" H 6850 2600 50  0001 C CNN
 F 1 "GND" H 6850 2700 50  0000 C CNN
 F 2 "" H 6850 2850 50  0001 C CNN
@@
 F 2 "Capacitors_SMD:C_0603" H 6588 4550 50  0001 C CNN
 F 3 "" H 6550 4700 50  0001 C CNN
-F 4 "CL10B104KC8NNNC" H 6550 4700 60  0001 C CNN "MFG"
+F 4 "ANY" H 6550 4700 60  0001 C CNN "MFG"
+F 5 "X7R" H 6550 4700 60  0001 C CNN "TempCo."
 	1    6550 4700
 	1    0    0    -1
@@
 F 2 "Capacitors_SMD:C_0603" H 6138 2500 50  0001 C CNN
 F 3 "" H 6100 2650 50  0001 C CNN
-F 4 "CL10B104KC8NNNC" H 6100 2650 60  0001 C CNN "MFG"
+F 4 "ANY" H 6100 2650 60  0001 C CNN "MFG"
+F 5 "X7R" H 6100 2650 60  0001 C CNN "TempCo."
 	1    6100 2650
 	0    1    1    0
@@
 Connection ~ 6300 2650
 $Comp
-L GND #PWR053
+L GND #PWR055
 U 1 1 5A8315FA
 P 5850 2700
-F 0 "#PWR053" H 5850 2450 50  0001 C CNN
+F 0 "#PWR055" H 5850 2450 50  0001 C CNN
 F 1 "GND" H 5850 2550 50  0000 C CNN
 F 2 "" H 5850 2700 50  0001 C CNN
@@
 F 2 "Resistors_SMD:R_1206" V 7680 3350 50  0001 C CNN
 F 3 "" H 7750 3350 50  0001 C CNN
-F 4 "KRL1632E-M-R010-F-T5" V 7750 3350 60  0001 C CNN "MFG"
+F 4 "ANY" V 7750 3350 60  0001 C CNN "MFG"
+F 5 "1%" V 7750 3350 60  0001 C CNN "Tol."
+F 6 "0.75W" V 7750 3350 60  0001 C CNN "Power"
 	1    7750 3350
 	1    0    0    -1
@@
 	5400 4400 5700 4400
 $Comp
-L GND #PWR054
+L GND #PWR056
 U 1 1 5A85F665
 P 2200 1550
-F 0 "#PWR054" H 2200 1300 50  0001 C CNN
+F 0 "#PWR056" H 2200 1300 50  0001 C CNN
 F 1 "GND" H 2200 1400 50  0000 C CNN
 F 2 "" H 2200 1550 50  0001 C CNN
@@
 $EndComp
 $Comp
-L +3V3 #PWR055
+L +3V3 #PWR057
 U 1 1 5A85F66B
 P 2100 1350
-F 0 "#PWR055" H 2100 1200 50  0001 C CNN
+F 0 "#PWR057" H 2100 1200 50  0001 C CNN
 F 1 "+3V3" H 2100 1490 50  0000 C CNN
 F 2 "" H 2100 1350 50  0001 C CNN
