File: Microcontroller.sch (KiCad schematic (older format))
At the start: 42 parts, among them J2 USB_OTG, J3 Conn_02x02, J4 JST_SMD_PH-04, J5 JST_SMD_PH-04, J7 GS3, J8 GS3, Q3 PMV50XPR, Q4 PMV50XPR, SW1 SW_Push, SW2 SW_Push, U1 AP2210N-3.3, U2 STM32L433CCT6, U8 TCAN330

Commit message: 0.2 HW files finalized and repo cleaned up.
-BOM is now up-to-date and available in .csv and .pdf formats
Parts:
- J3: MFG (none) -> M20-8750242
- J4, J5: MFG B4B-XH-A(LF)(SN) -> B4B-PH-SM4-TB(LF)(SN)
- J7, J8: MFG (none) -> SolderBridge
- TH2: MFG ERT-J1VR103J -> NCP18XH103J03RB
- U2: MFG (none) -> STM32L433CCT6
Changed lines of the file:
@@
 F 2 "Connectors_JST:JST_PH_B4B-PH-SM4-TB_04x2.00mm_Straight" H 8800 1350 50  0001 C CNN
 F 3 "" H 8800 1350 50  0001 C CNN
-F 4 "B4B-XH-A(LF)(SN)" H 8800 1350 60  0001 C CNN "MFG"
+F 4 "B4B-PH-SM4-TB(LF)(SN)" H 8800 1350 60  0001 C CNN "MFG"
 	1    8800 1350
 	1    0    0    -1
@@
 F 2 "Resistors_SMD:R_0603" H 10450 2800 50  0001 C CNN
 F 3 "" H 10450 2800 50  0001 C CNN
-F 4 "ERT-J1VR103J" V 10450 2750 60  0001 C CNN "MFG"
+F 4 "NCP18XH103J03RB" V 10450 2750 60  0001 C CNN "MFG"
 F 5 "5%" V 10450 2750 60  0001 C CNN "Tol."
 F 6 "4300K" V 10450 2750 60  0001 C CNN "B25/85"
@@
 F 2 "Connectors_JST:JST_PH_B4B-PH-SM4-TB_04x2.00mm_Straight" H 2450 1750 50  0001 C CNN
 F 3 "" H 2450 1750 50  0001 C CNN
-F 4 "B4B-XH-A(LF)(SN)" H 2450 1750 60  0001 C CNN "MFG"
+F 4 "B4B-PH-SM4-TB(LF)(SN)" H 2450 1750 60  0001 C CNN "MFG"
 	1    2450 1750
 	-1   0    0    1
@@
 F 2 "Housings_QFP:LQFP-48_7x7mm_Pitch0.5mm" H 5300 4000 60  0001 C CNN
 F 3 "" H 5300 4000 60  0001 C CNN
+F 4 "STM32L433CCT6" H 5500 4000 60  0001 C CNN "MFG"
 	1    5500 4000
 	1    0    0    -1
@@
 F 2 "Connectors:GS3" V 3338 1526 50  0001 C CNN
 F 3 "" H 3250 1600 50  0001 C CNN
+F 4 "SolderBridge" H 3250 1600 60  0001 C CNN "MFG"
 	1    3250 1600
 	-1   0    0    1
@@
 F 2 "Connectors:GS3" V 3338 1826 50  0001 C CNN
 F 3 "" H 3250 1900 50  0001 C CNN
+F 4 "SolderBridge" H 3250 1900 60  0001 C CNN "MFG"
 	1    3250 1900
 	-1   0    0    1
@@
 F 2 "Socket_Strips:Socket_Strip_Straight_2x02_Pitch2.54mm_SMD" H 1200 4900 50  0001 C CNN
 F 3 "" H 1200 4900 50  0001 C CNN
+F 4 "M20-8750242" H 1200 4900 60  0001 C CNN "MFG"
 	1    1200 4900
 	1    0    0    -1
